File: z80handheld.kicad_sch (KiCad schematic)
At the start: 133 parts, among them IC1 DS12885+, J1 Power, SW1 SW_Push_45deg, SW10 SW_Push_45deg, SW11 SW_Push_45deg, SW12 SW_Push_45deg, SW13 SW_Push_45deg, SW14 SW_Push_45deg, SW15 SW_Push_45deg, SW16 SW_Push_45deg, SW17 SW_Push_45deg, SW18 SW_Push_45deg, SW19 SW_Push_45deg, SW2 SW_Push_45deg, SW20 SW_Push_45deg, SW21 SW_Push_45deg, SW22 SW_Push_45deg, SW23 SW_Push_45deg, SW24 SW_Push_45deg, SW25 SW_Push_45deg, SW26 SW_Push_45deg, SW27 SW_Push_45deg, SW28 SW_Push_45deg, SW29 SW_Push_45deg, SW3 SW_Push_45deg, SW30 SW_Push_45deg, SW31 SW_Push_45deg, SW32 SW_Push_45deg, SW33 SW_Push_45deg, SW34 SW_Push_45deg, SW35 SW_Push_45deg, SW36 SW_Push_45deg, SW37 SW_Push_45deg, SW38 SW_Push_45deg, SW39 SW_Push_45deg, SW4 SW_Push_45deg, SW40 SW_Push_45deg, SW41 SW_Push_45deg, SW42 SW_Push_45deg, SW43 SW_Push_45deg, SW44 SW_Push_45deg, SW45 SW_Push_45deg, SW46 SW_Push_45deg, SW47 SW_Push_45deg, SW48 SW_Push_45deg, SW49 SW_Push_45deg, SW5 SW_Push_45deg, SW50 SW_Push_45deg, SW51 SW_Push_45deg, SW52 SW_Push_45deg, SW53 SW_Push_45deg, SW54 SW_Push_45deg, SW55 SW_Push_45deg, SW56 SW_Push_45deg, SW57 SW_Push_45deg, SW58 SW_Push_45deg, SW59 SW_Push_45deg, SW6 SW_Push_45deg, SW60 SW_Push_45deg, SW61 SW_Push_45deg, SW62 SW_Push_45deg, SW63 SW_Push_45deg, SW64 SW_Push_45deg, SW65 SW_Push, SW7 SW_Push_45deg, SW8 SW_Push_45deg, SW9 SW_Push_45deg, U1 74HC04, U10 Z84C00xxP, U11 74LS573 IO1, U12 SN76489AN, U13 74AHC1G02, U18 74AHCT1G32, U19 74AHCT1G32, U2 4068, U3 74HC04, U4 74154, U5 74LS573 IO0, U6 74LS573, U7 CY62256-70PC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

Commit message: Add files via upload
Parts:
- removed U13: 74AHC1G02, symbol 74xGxx:74AHC1G02
- removed U18, U19: 74AHCT1G32, Package_TO_SOT_SMD:SC-74A-5_1.55x2.9mm_P0.95mm, symbol 74xGxx:74AHCT1G32
- added U14: 74HCT02, Package_DIP:DIP-14_W7.62mm, symbol 74xx:74HCT02
- added unit 3 of U3
- added unit 7 of U3
- D1, D10, D11, D12, D13, D14, D15, D16, D17, D18, D19, D2, D20, D21, D22, D23, D24, D25, D26, D27, D28, D29, D3, D30, D31, D32, D33, D34, D35, D36, D37, D38, D39, D4, D5, D6, D7, D8, D9: footprint LED_SMD:LED_1206_3216Metric_Pad1.42x1.75mm_HandSolder -> LED_THT:LED_D5.0mm
- IC1: footprint DS12885:DIP1524W51P254L3175H508Q24N -> Library:DIP1524W51P254L3175H508Q24N
- RV1: footprint (none) -> Potentiometer_THT:Potentiometer_ACP_CA9-V10_Vertical
- U2: footprint PCM_Package_DIP_AKL:DIP-14_W7.62mm -> Package_DIP:DIP-14_W7.62mm
- U4: footprint PCM_Package_DIP_AKL:DIP-24_W7.62mm -> Package_DIP:DIP-24_W7.62mm
- U7, U8, U9: footprint Socket:DIP_Socket-28_W6.9mm_W7.62mm_W10.16mm_W12.7mm_W13.5mm_3M_228-4817-00-0602J -> Package_DIP:DIP-28_W15.24mm
Connections:
- net !MREQ: now also U14.12, U14.6, U14.9; no longer D5.2 (A), U1.4, U6.18 (Q1), U8.20 (~{CS})
- net !WR: now also U14.3
- net 5V: now also U14.14 (VCC), U3.14 (VCC); no longer U3.14 (VCC)
- net A15: now also U14.5
- net BANK_0: now also U7.20 (~{CS}), U3.6
- net GND: now also U14.7 (GND), U3.7 (GND); no longer U3.7 (GND)
- net IO2: now also U14.2
- net at U1.8: now also U9.20 (~{CS})
- net at U1.9: now also U14.4
- net at DS1.6 (E): now also U14.1
- net at U1.12: now also U14.11; no longer U7.20 (~{CS})
- new net: U1.4, U14.8
- new net: U14.13, U3.5
- new net: U14.10, U3.3
- new net BANK_1: D5.2 (A), U3.4, U6.18 (Q1), U8.20 (~{CS})
